File: ErgoChoco.kicad_pcb (KiCad board)
At the start: 2 copper layers, 129 parts, among them Q1 Q_NPN_BCE, U1 ProMicro

Commit message: added edge cuts, located PM
Parts:
- moved U1 6.47 mm to (148.4, 63.5)
Routing:
- net +5V: track 982.7 -> 942.9 mm
- net LEDGND: track 909.7 -> 897.1 mm
- net ROW3: track 169.8 -> 162.8 mm
Other:
- board outline added: 272 x 115.8 mm
Changed lines of the file:
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@@
   (general
     (thickness 1.6)
-    (drawings 0)
-    (tracks 524)
+    (drawings 24)
+    (tracks 520)
     (zones 0)
     (modules 129)
@@
   )
   (module Keebio-Parts:ArduinoProMicro (layer B.Cu)
-    (at 148.43125 70 270)
+    (at 148.43125 63.53 270)
     (fp_text reference U1 (at 0 -1.625 270) (layer B.SilkS) hide
       (effects (font (size 1.27 1.524) (thickness 0.2032)) (justify mirror))
@@
     )
   )
+  (gr_arc (start 15.43125 105.4971) (end 12.43125 105.4971) (angle -65) (layer Edge.Cuts) (width 0.05))
+  (gr_arc (start 129.09633 158.5) (end 129.09633 161.5) (angle 25) (layer Edge.Cuts) (width 0.05))
+  (gr_arc (start 167.76617 158.5) (end 167.76617 161.5) (angle -25) (layer Edge.Cuts) (width 0.05))
+  (gr_arc (start 281.43125 105.4971) (end 284.43125 105.4971) (angle 65) (layer Edge.Cuts) (width 0.05))
+  (gr_arc (start 281.43125 52.5) (end 281.43125 49.5) (angle 90) (layer Edge.Cuts) (width 0.05))
+  (gr_arc (start 165.92389 46.5) (end 165.92389 49.5) (angle 45) (layer Edge.Cuts) (width 0.05))
+  (gr_arc (start 159.68861 48.75) (end 159.68861 45.75) (angle 45) (layer Edge.Cuts) (width 0.05))
+  (gr_arc (start 137.17389 48.75) (end 137.17389 45.75) (angle -45) (layer Edge.Cuts) (width 0.05))
+  (gr_arc (start 130.93861 46.5) (end 133.05993 48.62132) (angle 45) (layer Edge.Cuts) (width 0.05))
+  (gr_arc (start 15.43125 52.5) (end 15.43125 49.5) (angle -90) (layer Edge.Cuts) (width 0.05))
+  (gr_line (start 12.43125 52.5) (end 12.43125 105.4971) (layer Edge.Cuts) (width 0.05))
+  (gr_line (start 14.1634 108.21602) (end 127.82848 161.21892) (layer Edge.Cuts) (width 0.05))
+  (gr_line (start 129.09633 161.5) (end 167.76617 161.5) (layer Edge.Cuts) (width 0.05))
+  (gr_line (start 282.6991 108.21602) (end 169.03402 161.21892) (layer Edge.Cuts) (width 0.05))
+  (gr_line (start 284.43125 52.5) (end 284.43125 105.4971) (layer Edge.Cuts) (width 0.05))
+  (gr_line (start 165.92389 49.5) (end 281.43125 49.5) (layer Edge.Cuts) (width 0.05))
+  (gr_line (start 161.80993 46.62868) (end 163.80257 48.62132) (layer Edge.Cuts) (width 0.05))
+  (gr_line (start 154.43125 45.75) (end 159.68861 45.75) (layer Edge.Cuts) (width 0.05))
+  (gr_line (start 154.43125 45.75) (end 154.43125 77.75) (layer Edge.Cuts) (width 0.05))
+  (gr_line (start 142.43125 77.75) (end 154.43125 77.75) (layer Edge.Cuts) (width 0.05))
+  (gr_line (start 142.43125 45.75) (end 142.43125 77.75) (layer Edge.Cuts) (width 0.05))
+  (gr_line (start 137.17389 45.75) (end 142.43125 45.75) (layer Edge.Cuts) (width 0.05))
+  (gr_line (start 133.05993 48.62132) (end 135.05257 46.62868) (layer Edge.Cuts) (width 0.05))
+  (gr_line (start 15.43125 49.5) (end 130.93861 49.5) (layer Edge.Cuts) (width 0.05))
   (via (at 214.484115 88.78212) (size 0.8) (drill 0.4) (layers F.Cu B.Cu) (net 105))
   (via (at 236.35356 87.65259) (size 0.8) (drill 0.4) (layers F.Cu B.Cu) (net 17))
@@
   (segment (start 118.584302 149.904847) (end 114.56752 153.92163) (width 0.381) (layer B.Cu) (net 2))
   (segment (start 98.66123 144.73813) (end 114.56752 153.92163) (width 0.381) (layer F.Cu) (net 2))
-  (segment (start 114.56752 153.92163) (end 134.66488 165.52485) (width 0.381) (layer F.Cu) (net 2))
   (via (at 211.61193 135.82431) (size 0.8) (drill 0.4) (layers F.Cu B.Cu) (net 2))
   (segment (start 210.413745 131.352623) (end 211.61193 135.82431) (width 0.381) (layer B.Cu) (net 2))
@@
   (segment (start 176.484297 151.700898) (end 179.27655 154.49315) (width 0.381) (layer B.Cu) (net 2))
   (segment (start 195.48304 145.13633) (end 179.27655 154.49315) (width 0.381) (layer F.Cu) (net 2))
-  (segment (start 179.27655 154.49315) (end 164.9666 162.755) (width 0.381) (layer F.Cu) (net 2))
   (segment (start 41.730474 60.711069) (end 42.369404 65.341482) (width 0.254) (layer B.Cu) (net 3))
   (segment (start 243.83118 76.45636) (end 231.436 69.3) (width 0.254) (layer F.Cu) (net 4))
@@
   (segment (start 108.72991 148.17977) (end 125.7257 157.9923) (width 0.254) (layer F.Cu) (net 42))
   (segment (start 128.157885 155.560115) (end 125.7257 157.9923) (width 0.254) (layer B.Cu) (net 42))
-  (segment (start 125.7257 157.9923) (end 131.85665 161.532) (width 0.254) (layer F.Cu) (net 42))
   (via (at 220.71194 128.38688) (size 0.8) (drill 0.4) (layers F.Cu B.Cu) (net 42))
   (segment (start 219.915404 125.412518) (end 220.71194 128.38688) (width 0.254) (layer B.Cu) (net 42))
@@
   (segment (start 123.217913 154.586913) (end 121.34881 156.45601) (width 0.381) (layer B.Cu) (net 105))
   (segment (start 104.96997 146.99968) (end 121.34881 156.45601) (width 0.381) (layer F.Cu) (net 105))
-  (segment (start 121.34881 156.45601) (end 132.20207 162.72214) (width 0.381) (layer F.Cu) (net 105))
   (segment (start 216.805555 129.678357) (end 217.26889 131.40755) (width 0.381) (layer B.Cu) (net 105))
   (via (at 217.26889 131.40755) (size 0.8) (drill 0.4) (layers F.Cu B.Cu) (net 105))
