File: ErgoChoco.kicad_pcb (KiCad board)
At the start: 2 copper layers, 272 x 115.8 mm, 129 parts, among them Q1 Q_NPN_BCE, U1 ProMicro

Commit message: finished routing, added mounting holes
Parts:
- added J1: Conn_01x03, Connector_PinHeader_2.54mm:PinHeader_1x03_P2.54mm_Vertical, F.Cu at (17.8, 54.6)
- added REF**: PTH_2.2_4, Choco617_parts:PTH_2.2_4, F.Cu at (176.3, 55.2)
- added REF**: PTH_2.2_4, Choco617_parts:PTH_2.2_4, F.Cu at (249.2, 118.5)
- added REF**: PTH_2.2_4, Choco617_parts:PTH_2.2_4, F.Cu at (173.8, 130.8)
- added REF**: PTH_2.2_4, Choco617_parts:PTH_2.2_4, F.Cu at (279.1, 67.2)
- added REF**: PTH_2.2_4, Choco617_parts:PTH_2.2_4, F.Cu at (123.1, 130.8)
- added REF**: PTH_2.2_4, Choco617_parts:PTH_2.2_4, F.Cu at (47.7, 118.5)
- added REF**: PTH_2.2_4, Choco617_parts:PTH_2.2_4, F.Cu at (120.5, 55.2)
- added REF**: PTH_2.2_4, Choco617_parts:PTH_2.2_4, F.Cu at (17.8, 67.2)
- added SW1: SW_Push, random-keyboard-parts:SKQG-1155865, F.Cu at (130.2, 55.6)
- NPNR1: moved to B.Cu
- Q1: footprint digikey-footprints:Trans_SOT-223-4 -> digikey-footprints:SOT-23-3; moved to B.Cu
- moved Q1 91.4 mm to (148.4, 94.6)
- moved NPNR1 86.3 mm to (147.5, 82.7), turned to 90 degrees
- moved D6 3.03 mm to (136.7, 82.7)
Connections:
- U1 pad 1: Net-(U1-Pad1) -> COL11
- U1 pad 10: Net-(U1-Pad10) -> ROW1
- U1 pad 11: Net-(U1-Pad11) -> ROW2
- U1 pad 12: Net-(U1-Pad12) -> LEDPWM
- U1 pad 13: Net-(U1-Pad13) -> ROW3
- U1 pad 14: Net-(U1-Pad14) -> COL5
- U1 pad 15: Net-(U1-Pad15) -> COL4
- U1 pad 16: Net-(U1-Pad16) -> COL3
- U1 pad 17: Net-(U1-Pad17) -> COL2
- U1 pad 18: Net-(U1-Pad18) -> COL1
- U1 pad 19: Net-(U1-Pad19) -> COL0
- U1 pad 2: Net-(U1-Pad2) -> COL10
- U1 pad 21: Net-(U1-Pad21) -> +5V
- U1 pad 23: Net-(U1-Pad23) -> GND
- U1 pad 3: Net-(U1-Pad3) -> GND
- U1 pad 4: Net-(U1-Pad4) -> GND
- U1 pad 5: Net-(U1-Pad5) -> COL9
- U1 pad 6: Net-(U1-Pad6) -> COL8
- U1 pad 7: Net-(U1-Pad7) -> COL7
- U1 pad 8: Net-(U1-Pad8) -> COL6
- U1 pad 9: Net-(U1-Pad9) -> ROW0
Routing:
- net +5V: track 942.9 -> 1337.9 mm, vias 36 -> 46
- net LEDGND: track 897.1 -> 1125.5 mm, vias 39 -> 46
- net Net-(J1-Pad2): track 0.00 -> 132.1 mm
- net COL0: track 38.0 -> 165.0 mm
- net COL1: track 38.0 -> 148.2 mm
- net ROW2: track 264.1 -> 374.2 mm, vias 11 -> 13
- net COL11: track 38.0 -> 146.9 mm
- net ROW3: track 162.8 -> 261.7 mm, vias 6 -> 7
- net COL10: track 38.0 -> 131.8 mm
- net ROW1: track 264.1 -> 348.5 mm, vias 11 -> 13
- net COL2: track 38.0 -> 120.4 mm
- net COL9: track 38.0 -> 109.3 mm
- net COL3: track 66.7 -> 128.0 mm
- net ROW0: track 263.8 -> 322.4 mm, vias 11 -> 13
- net COL4: track 63.2 -> 105.1 mm
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- added copper zone on B.Cu, net GND
- added copper zone on F.Cu, net GND
Other:
- outline, holes or cut-outs redrawn
- board text added: "+5V"
- board text added: "ErgoChoco v1.0 designed by u/Choco617 repo: https://github.com/ Choco617/ErgoChoco-PCB"
- board text added: "F4"
- board text added: "GND"
